File: Power_supply2.sch (EAGLE design)
At the start: 34 parts, among them IC1 7808T, IC2 7812T, IC3 7808T, IC4 7808T, IC5 7808T, IC6 7808T

Commit message: Finished BRD
Parts:
- renumbered JP2 to 1, JP3 to 3, JP4 to 4, JP5 to 5, JP6 to 6
Changed lines of the file:
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@@
 <part name="C18" library="resistor" deviceset="C-EU" device="C0805" value="2n2"/>
 <part name="TRANS" library="pinhead" deviceset="PINHD-1X2" device=""/>
-<part name="JP2" library="pinhead" deviceset="PINHD-1X2" device=""/>
-<part name="JP3" library="pinhead" deviceset="PINHD-1X2" device=""/>
-<part name="JP4" library="pinhead" deviceset="PINHD-1X2" device=""/>
-<part name="JP5" library="pinhead" deviceset="PINHD-1X2" device=""/>
-<part name="JP6" library="pinhead" deviceset="PINHD-1X2" device=""/>
+<part name="1" library="pinhead" deviceset="PINHD-1X2" device=""/>
+<part name="3" library="pinhead" deviceset="PINHD-1X2" device=""/>
+<part name="4" library="pinhead" deviceset="PINHD-1X2" device=""/>
+<part name="5" library="pinhead" deviceset="PINHD-1X2" device=""/>
+<part name="6" library="pinhead" deviceset="PINHD-1X2" device=""/>
 </parts>
 <sheets>
@@
 <instance part="C18" gate="G$1" x="5.08" y="-7.62" rot="R90"/>
 <instance part="TRANS" gate="G$1" x="-27.94" y="20.32" rot="R180"/>
-<instance part="JP2" gate="G$1" x="180.34" y="55.88"/>
-<instance part="JP3" gate="G$1" x="180.34" y="33.02"/>
-<instance part="JP4" gate="G$1" x="180.34" y="7.62"/>
-<instance part="JP5" gate="G$1" x="180.34" y="-17.78"/>
-<instance part="JP6" gate="G$1" x="180.34" y="-40.64"/>
+<instance part="1" gate="G$1" x="180.34" y="55.88"/>
+<instance part="3" gate="G$1" x="180.34" y="33.02"/>
+<instance part="4" gate="G$1" x="180.34" y="7.62"/>
+<instance part="5" gate="G$1" x="180.34" y="-17.78"/>
+<instance part="6" gate="G$1" x="180.34" y="-40.64"/>
 </instances>
 <busses>
@@
 <wire x1="165.1" y1="12.7" x2="165.1" y2="10.16" width="0.1524" layer="91"/>
 <junction x="157.48" y="12.7"/>
-<pinref part="JP4" gate="G$1" pin="1"/>
+<pinref part="4" gate="G$1" pin="1"/>
 <wire x1="177.8" y1="10.16" x2="175.26" y2="10.16" width="0.1524" layer="91"/>
 <wire x1="175.26" y1="10.16" x2="175.26" y2="12.7" width="0.1524" layer="91"/>
@@
 <wire x1="167.64" y1="-12.7" x2="167.64" y2="-15.24" width="0.1524" layer="91"/>
 <junction x="160.02" y="-12.7"/>
-<pinref part="JP5" gate="G$1" pin="1"/>
+<pinref part="5" gate="G$1" pin="1"/>
 <wire x1="177.8" y1="-15.24" x2="175.26" y2="-15.24" width="0.1524" layer="91"/>
 <wire x1="175.26" y1="-15.24" x2="175.26" y2="-12.7" width="0.1524" layer="91"/>
@@
 <wire x1="157.48" y1="58.42" x2="157.48" y2="60.96" width="0.1524" layer="91"/>
 <junction x="157.48" y="60.96"/>
-<pinref part="JP2" gate="G$1" pin="1"/>
+<pinref part="1" gate="G$1" pin="1"/>
 <wire x1="177.8" y1="58.42" x2="175.26" y2="58.42" width="0.1524" layer="91"/>
 <wire x1="175.26" y1="58.42" x2="175.26" y2="60.96" width="0.1524" layer="91"/>
@@
 <wire x1="165.1" y1="38.1" x2="165.1" y2="35.56" width="0.1524" layer="91"/>
 <junction x="157.48" y="38.1"/>
-<pinref part="JP3" gate="G$1" pin="1"/>
+<pinref part="3" gate="G$1" pin="1"/>
 <wire x1="177.8" y1="35.56" x2="175.26" y2="35.56" width="0.1524" layer="91"/>
 <wire x1="175.26" y1="35.56" x2="175.26" y2="38.1" width="0.1524" layer="91"/>
@@
 <wire x1="167.64" y1="-35.56" x2="167.64" y2="-38.1" width="0.1524" layer="91"/>
 <junction x="160.02" y="-35.56"/>
-<pinref part="JP6" gate="G$1" pin="1"/>
+<pinref part="6" gate="G$1" pin="1"/>
 <wire x1="177.8" y1="-38.1" x2="175.26" y2="-38.1" width="0.1524" layer="91"/>
 <wire x1="175.26" y1="-38.1" x2="175.26" y2="-35.56" width="0.1524" layer="91"/>
@@
 <wire x1="30.48" y1="-10.16" x2="33.02" y2="-10.16" width="0.1524" layer="91"/>
 <junction x="33.02" y="-10.16"/>
-<pinref part="JP2" gate="G$1" pin="2"/>
+<pinref part="1" gate="G$1" pin="2"/>
 <wire x1="177.8" y1="55.88" x2="175.26" y2="55.88" width="0.1524" layer="91"/>
 <wire x1="175.26" y1="55.88" x2="175.26" y2="48.26" width="0.1524" layer="91"/>
 <wire x1="175.26" y1="48.26" x2="165.1" y2="48.26" width="0.1524" layer="91"/>
 <junction x="165.1" y="48.26"/>
-<pinref part="JP3" gate="G$1" pin="2"/>
+<pinref part="3" gate="G$1" pin="2"/>
 <wire x1="177.8" y1="33.02" x2="175.26" y2="33.02" width="0.1524" layer="91"/>
 <wire x1="175.26" y1="33.02" x2="175.26" y2="22.86" width="0.1524" layer="91"/>
 <wire x1="175.26" y1="22.86" x2="165.1" y2="22.86" width="0.1524" layer="91"/>
 <junction x="165.1" y="22.86"/>
-<pinref part="JP4" gate="G$1" pin="2"/>
+<pinref part="4" gate="G$1" pin="2"/>
 <wire x1="177.8" y1="7.62" x2="175.26" y2="7.62" width="0.1524" layer="91"/>
 <wire x1="175.26" y1="7.62" x2="175.26" y2="0" width="0.1524" layer="91"/>
 <wire x1="175.26" y1="0" x2="165.1" y2="0" width="0.1524" layer="91"/>
 <junction x="165.1" y="0"/>
-<pinref part="JP5" gate="G$1" pin="2"/>
+<pinref part="5" gate="G$1" pin="2"/>
 <wire x1="177.8" y1="-17.78" x2="175.26" y2="-17.78" width="0.1524" layer="91"/>
 <wire x1="175.26" y1="-17.78" x2="175.26" y2="-25.4" width="0.1524" layer="91"/>
 <wire x1="175.26" y1="-25.4" x2="167.64" y2="-25.4" width="0.1524" layer="91"/>
 <junction x="167.64" y="-25.4"/>
-<pinref part="JP6" gate="G$1" pin="2"/>
+<pinref part="6" gate="G$1" pin="2"/>
 <wire x1="177.8" y1="-40.64" x2="175.26" y2="-40.64" width="0.1524" layer="91"/>
 <wire x1="175.26" y1="-40.64" x2="175.26" y2="-50.8" width="0.1524" layer="91"/>

Commit message: Modofied SCH & BRD
Parts:
- removed C10, C11, C12, C13: 10u, resistor:CPOL-EUE3.5-8
- removed C2: 100u, resistor:CPOL-EUE5-13
- added C19, C20, C21, C22, C23: 10u, resistor:CPOL-EUCT7343
- C3: value 100u -> 1000u
- C9: value 10u -> 100u; device resistor:CPOL-EUE3.5-8 -> resistor:CPOL-EUE2.5-6
Connections:
- net GND: now also C19.-, C20.-, C21.-, C22.-, C23.-; no longer C10.-, C11.-, C12.-, C13.-, C2.-
- net N$2: now also C21.+; no longer C11.+
- net N$3: now also C22.+; no longer C12.+
- net N$4: now also C19.+; no longer C9.+
- net N$5: now also C9.+; no longer C2.+
- net N$6: now also C20.+; no longer C10.+
- net N$7: now also C23.+; no longer C13.+
Other:
- moved on the sheet: C9
Changed lines of the file:
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@@
 <part name="IC6" library="linear" deviceset="78*" device="T" technology="08"/>
 <part name="C1" library="resistor" deviceset="C-EU" device="C0805" value="100n"/>
-<part name="C2" library="resistor" deviceset="CPOL-EU" device="E5-13" value="100u"/>
-<part name="C3" library="resistor" deviceset="CPOL-EU" device="E5-13" value="100u"/>
+<part name="C3" library="resistor" deviceset="CPOL-EU" device="E5-13" value="1000u"/>
 <part name="C4" library="resistor" deviceset="C-EU" device="C0805" value="100n"/>
 <part name="C5" library="resistor" deviceset="C-EU" device="C0805" value="100n"/>
@@
 <part name="C7" library="resistor" deviceset="C-EU" device="C0805" value="100n"/>
 <part name="C8" library="resistor" deviceset="C-EU" device="C0805" value="100n"/>
-<part name="C9" library="resistor" deviceset="CPOL-EU" device="E3.5-8" value="10u"/>
-<part name="C10" library="resistor" deviceset="CPOL-EU" device="E3.5-8" value="10u"/>
-<part name="C11" library="resistor" deviceset="CPOL-EU" device="E3.5-8" value="10u"/>
-<part name="C12" library="resistor" deviceset="CPOL-EU" device="E3.5-8" value="10u"/>
-<part name="C13" library="resistor" deviceset="CPOL-EU" device="E3.5-8" value="10u"/>
 <part name="C14" library="resistor" deviceset="C-EU" device="C0805" value="100n"/>
 <part name="GND1" library="supply1" deviceset="GND" device=""/>
@@
 <part name="5" library="pinhead" deviceset="PINHD-1X2" device=""/>
 <part name="6" library="pinhead" deviceset="PINHD-1X2" device=""/>
+<part name="C19" library="resistor" deviceset="CPOL-EU" device="CT7343" value="10u"/>
+<part name="C20" library="resistor" deviceset="CPOL-EU" device="CT7343" value="10u"/>
+<part name="C21" library="resistor" deviceset="CPOL-EU" device="CT7343" value="10u"/>
+<part name="C22" library="resistor" deviceset="CPOL-EU" device="CT7343" value="10u"/>
+<part name="C23" library="resistor" deviceset="CPOL-EU" device="CT7343" value="10u"/>
+<part name="C9" library="resistor" deviceset="CPOL-EU" device="E2.5-6" value="100u"/>
 </parts>
 <sheets>
@@
 <instance part="IC6" gate="A1" x="139.7" y="-35.56"/>
 <instance part="C1" gate="G$1" x="91.44" y="-2.54"/>
-<instance part="C2" gate="G$1" x="83.82" y="-2.54"/>
 <instance part="C3" gate="G$1" x="33.02" y="-2.54"/>
 <instance part="C4" gate="G$1" x="165.1" y="55.88"/>
@@
 <instance part="C7" gate="G$1" x="167.64" y="-17.78"/>
 <instance part="C8" gate="G$1" x="167.64" y="-40.64"/>
-<instance part="C9" gate="G$1" x="157.48" y="55.88"/>
-<instance part="C10" gate="G$1" x="157.48" y="33.02"/>
-<instance part="C11" gate="G$1" x="157.48" y="7.62"/>
-<instance part="C12" gate="G$1" x="160.02" y="-17.78"/>
-<instance part="C13" gate="G$1" x="160.02" y="-40.64"/>
 <instance part="C14" gate="G$1" x="43.18" y="-2.54"/>
 <instance part="GND1" gate="1" x="60.96" y="-53.34"/>
@@
 <instance part="5" gate="G$1" x="180.34" y="-17.78"/>
 <instance part="6" gate="G$1" x="180.34" y="-40.64"/>
+<instance part="C19" gate="G$1" x="157.48" y="55.88"/>
+<instance part="C20" gate="G$1" x="157.48" y="33.02"/>
+<instance part="C21" gate="G$1" x="157.48" y="7.62"/>
+<instance part="C22" gate="G$1" x="160.02" y="-17.78"/>
+<instance part="C23" gate="G$1" x="160.02" y="-40.64"/>
+<instance part="C9" gate="G$1" x="83.82" y="-2.54"/>
 </instances>
 <busses>
@@
 <wire x1="111.76" y1="-35.56" x2="111.76" y2="-12.7" width="0.1524" layer="91"/>
 <junction x="111.76" y="-12.7"/>
-<pinref part="C2" gate="G$1" pin="+"/>
 <wire x1="83.82" y1="0" x2="83.82" y2="5.08" width="0.1524" layer="91"/>
 <junction x="83.82" y="5.08"/>
@@
 <wire x1="91.44" y1="0" x2="91.44" y2="5.08" width="0.1524" layer="91"/>
 <junction x="91.44" y="5.08"/>
+<pinref part="C9" gate="G$1" pin="+"/>
 </segment>
 </net>
@@
 <segment>
 <pinref part="IC4" gate="A1" pin="VO"/>
-<pinref part="C11" gate="G$1" pin="+"/>
 <wire x1="149.86" y1="12.7" x2="157.48" y2="12.7" width="0.1524" layer="91"/>
 <wire x1="157.48" y1="12.7" x2="157.48" y2="10.16" width="0.1524" layer="91"/>
@@
 <wire x1="175.26" y1="12.7" x2="165.1" y2="12.7" width="0.1524" layer="91"/>
 <junction x="165.1" y="12.7"/>
+<pinref part="C21" gate="G$1" pin="+"/>
 </segment>
 </net>
@@
 <segment>
 <pinref part="IC5" gate="A1" pin="VO"/>
-<pinref part="C12" gate="G$1" pin="+"/>
 <wire x1="149.86" y1="-12.7" x2="160.02" y2="-12.7" width="0.1524" layer="91"/>
 <wire x1="160.02" y1="-12.7" x2="160.02" y2="-15.24" width="0.1524" layer="91"/>
@@
 <wire x1="175.26" y1="-12.7" x2="167.64" y2="-12.7" width="0.1524" layer="91"/>
 <junction x="167.64" y="-12.7"/>
+<pinref part="C22" gate="G$1" pin="+"/>
 </segment>
 </net>
@@
 <wire x1="157.48" y1="60.96" x2="165.1" y2="60.96" width="0.1524" layer="91"/>
 <wire x1="165.1" y1="60.96" x2="165.1" y2="58.42" width="0.1524" layer="91"/>
-<pinref part="C9" gate="G$1" pin="+"/>
 <wire x1="157.48" y1="58.42" x2="157.48" y2="60.96" width="0.1524" layer="91"/>
 <junction x="157.48" y="60.96"/>
@@
 <wire x1="175.26" y1="60.96" x2="165.1" y2="60.96" width="0.1524" layer="91"/>
 <junction x="165.1" y="60.96"/>
+<pinref part="C19" gate="G$1" pin="+"/>
 </segment>
 </net>
@@
 <segment>
 <pinref part="IC3" gate="A1" pin="VO"/>
-<pinref part="C10" gate="G$1" pin="+"/>
 <wire x1="149.86" y1="38.1" x2="157.48" y2="38.1" width="0.1524" layer="91"/>
 <wire x1="157.48" y1="38.1" x2="157.48" y2="35.56" width="0.1524" layer="91"/>
@@
 <wire x1="175.26" y1="38.1" x2="165.1" y2="38.1" width="0.1524" layer="91"/>
 <junction x="165.1" y="38.1"/>
+<pinref part="C20" gate="G$1" pin="+"/>
 </segment>
 </net>
@@
 <segment>
 <pinref part="IC6" gate="A1" pin="VO"/>
-<pinref part="C13" gate="G$1" pin="+"/>
 <wire x1="149.86" y1="-35.56" x2="160.02" y2="-35.56" width="0.1524" layer="91"/>
 <wire x1="160.02" y1="-35.56" x2="160.02" y2="-38.1" width="0.1524" layer="91"/>
@@
 <wire x1="175.26" y1="-35.56" x2="167.64" y2="-35.56" width="0.1524" layer="91"/>
 <junction x="167.64" y="-35.56"/>
+<pinref part="C23" gate="G$1" pin="+"/>
 </segment>
 </net>
@@
 <junction x="124.46" y="-50.8"/>
 <wire x1="60.96" y1="-50.8" x2="124.46" y2="-50.8" width="0.1524" layer="91"/>
-<pinref part="C11" gate="G$1" pin="-"/>
 <wire x1="157.48" y1="2.54" x2="157.48" y2="0" width="0.1524" layer="91"/>
 <wire x1="157.48" y1="0" x2="139.7" y2="0" width="0.1524" layer="91"/>
@@
 <wire x1="165.1" y1="0" x2="157.48" y2="0" width="0.1524" layer="91"/>
 <junction x="157.48" y="0"/>
-<pinref part="C9" gate="G$1" pin="-"/>
 <wire x1="157.48" y1="50.8" x2="157.48" y2="48.26" width="0.1524" layer="91"/>
 <wire x1="157.48" y1="48.26" x2="139.7" y2="48.26" width="0.1524" layer="91"/>
@@
 <wire x1="165.1" y1="48.26" x2="157.48" y2="48.26" width="0.1524" layer="91"/>
 <junction x="157.48" y="48.26"/>
-<pinref part="C10" gate="G$1" pin="-"/>
 <wire x1="157.48" y1="27.94" x2="157.48" y2="22.86" width="0.1524" layer="91"/>
 <wire x1="157.48" y1="22.86" x2="139.7" y2="22.86" width="0.1524" layer="91"/>
@@
 <wire x1="165.1" y1="22.86" x2="157.48" y2="22.86" width="0.1524" layer="91"/>
 <junction x="157.48" y="22.86"/>
-<pinref part="C12" gate="G$1" pin="-"/>
 <wire x1="139.7" y1="-25.4" x2="160.02" y2="-25.4" width="0.1524" layer="91"/>
 <wire x1="160.02" y1="-25.4" x2="160.02" y2="-22.86" width="0.1524" layer="91"/>
@@
 <wire x1="167.64" y1="-25.4" x2="167.64" y2="-22.86" width="0.1524" layer="91"/>
 <junction x="160.02" y="-25.4"/>
-<pinref part="C13" gate="G$1" pin="-"/>
 <wire x1="160.02" y1="-45.72" x2="160.02" y2="-50.8" width="0.1524" layer="91"/>
 <wire x1="160.02" y1="-50.8" x2="139.7" y2="-50.8" width="0.1524" layer="91"/>
@@
 <wire x1="43.18" y1="-10.16" x2="60.96" y2="-10.16" width="0.1524" layer="91"/>
 <junction x="60.96" y="-10.16"/>
-<pinref part="C2" gate="G$1" pin="-"/>
 <wire x1="60.96" y1="-10.16" x2="83.82" y2="-10.16" width="0.1524" layer="91"/>
 <wire x1="83.82" y1="-10.16" x2="83.82" y2="-7.62" width="0.1524" layer="91"/>
@@
 <wire x1="175.26" y1="-50.8" x2="167.64" y2="-50.8" width="0.1524" layer="91"/>
 <junction x="167.64" y="-50.8"/>
-</segment>
-</net>
+<pinref part="C19" gate="G$1" pin="-"/>
+<pinref part="C20" gate="G$1" pin="-"/>
+<pinref part="C21" gate="G$1" pin="-"/>
+<pinref part="C22" gate="G$1" pin="-"/>
+<pinref part="C23" gate="G$1" pin="-"/>
+<pinref part="C9" gate="G$1" pin="-"/>
+</segment>
+</net>
